File: V1/Relay-24v-4ch-V1.kicad_sch (KiCad schematic)
At the start: 25 parts, among them J1 Conn_01x05, J3 OUT1, J3 OUT2, J3 OUT3, J3 OUT4, K1 G5PZ-1A

Commit message: Update board images
Connections:
- net +24V: now also J1.5 (Pin_5); no longer J1.1 (Pin_1)
- net at D14.1 (K), D15.2 (A), K1.4: now also J1.1 (Pin_1); no longer J1.5 (Pin_5)
- net at D14.1 (K), D15.2 (A), K1.4: now also J1.2 (Pin_2); no longer J1.4 (Pin_4)
- net at D14.1 (K), D15.2 (A), K1.4: now also J1.4 (Pin_4); no longer J1.2 (Pin_2)
Other:
- moved on the sheet: J1
Changed lines of the file:
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@@
     )
   )
-  (symbol (lib_id "Connector_Generic:Conn_01x05") (at 38.1 88.9 0) (mirror y) (unit 1)
-    (in_bom yes) (on_board yes) (dnp no) (fields_autoplaced)
-    (property "Reference" "J1" (at 38.1 78.74 0)
+  (symbol (lib_id "Connector_Generic:Conn_01x05") (at 38.1 88.9 180) (unit 1)
+    (in_bom yes) (on_board yes) (dnp no)
+    (property "Reference" "J1" (at 38.1 77.47 0)
       (effects (font (size 1.27 1.27)))
     )
-    (property "Value" "Conn_01x05" (at 38.1 81.28 0)
+    (property "Value" "Conn_01x05" (at 38.1 80.01 0)
       (effects (font (size 1.27 1.27)))
     )

Commit message: Adjustments for fabrication
Parts:
- D14: value BLUE/0603 -> GREEN/0603; LCSC Part # C72041 -> C72043; Mfr PN 19-217/BHC-ZL1M2RY/3T -> 19-217/GHC-YR1S2/3T; Vendor PN C72041 -> C72043
- J1: JLCPCB BOM (none) -> 1; LCSC Part # (none) -> C2898747; Mfr (none) -> Dibo; Mfr PN (none) -> DB141V-2.54-5P; Vendor (none) -> JLCPCB; Vendor PN (none) -> C2898747
Changed lines of the file:
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@@
       (effects (font (size 1.27 1.27)) (justify left))
     )
-    (property "Value" "BLUE/0603" (at 184.15 118.11 90)
+    (property "Value" "GREEN/0603" (at 184.15 118.11 90)
       (effects (font (size 1.27 1.27)) (justify left))
     )
@@
       (effects (font (size 1.27 1.27)) hide)
     )
-    (property "Mfr PN" "19-217/BHC-ZL1M2RY/3T" (at 186.69 118.11 0)
+    (property "Mfr PN" "19-217/GHC-YR1S2/3T" (at 186.69 118.11 0)
       (effects (font (size 1.27 1.27)) hide)
     )
@@
       (effects (font (size 1.27 1.27)) hide)
     )
-    (property "Vendor PN" "C72041" (at 186.69 118.11 0)
-      (effects (font (size 1.27 1.27)) hide)
-    )
-    (property "LCSC Part #" "C72041" (at 184.15 120.65 90)
+    (property "Vendor PN" "C72043" (at 186.69 118.11 0)
+      (effects (font (size 1.27 1.27)) hide)
+    )
+    (property "LCSC Part #" "C72043" (at 184.15 120.65 90)
       (effects (font (size 1.27 1.27)) (justify left))
     )
@@
     )
     (property "Datasheet" "~" (at 38.1 88.9 0)
+      (effects (font (size 1.27 1.27)) hide)
+    )
+    (property "Case" "~" (at 38.1 88.9 0)
+      (effects (font (size 1.27 1.27)) hide)
+    )
+    (property "JLCPCB BOM" "1" (at 38.1 88.9 0)
+      (effects (font (size 1.27 1.27)) hide)
+    )
+    (property "LCSC Part #" "C2898747" (at 38.1 88.9 0)
+      (effects (font (size 1.27 1.27)) hide)
+    )
+    (property "Mfr" "Dibo" (at 38.1 88.9 0)
+      (effects (font (size 1.27 1.27)) hide)
+    )
+    (property "Mfr PN" "DB141V-2.54-5P" (at 38.1 88.9 0)
+      (effects (font (size 1.27 1.27)) hide)
+    )
+    (property "Technology" "~" (at 38.1 88.9 0)
+      (effects (font (size 1.27 1.27)) hide)
+    )
+    (property "Vendor" "JLCPCB" (at 38.1 88.9 0)
+      (effects (font (size 1.27 1.27)) hide)
+    )
+    (property "Vendor PN" "C2898747" (at 38.1 88.9 0)
       (effects (font (size 1.27 1.27)) hide)
     )
@@
       (effects (font (size 1.27 1.27)) (justify left))
     )
-    (property "Value" "BLUE/0603" (at 81.28 118.11 90)
+    (property "Value" "GREEN/0603" (at 81.28 118.11 90)
       (effects (font (size 1.27 1.27)) (justify left))
     )
@@
       (effects (font (size 1.27 1.27)) hide)
     )
-    (property "Mfr PN" "19-217/BHC-ZL1M2RY/3T" (at 83.82 118.11 0)
+    (property "Mfr PN" "19-217/GHC-YR1S2/3T" (at 83.82 118.11 0)
       (effects (font (size 1.27 1.27)) hide)
     )
@@
       (effects (font (size 1.27 1.27)) hide)
     )
-    (property "Vendor PN" "C72041" (at 83.82 118.11 0)
-      (effects (font (size 1.27 1.27)) hide)
-    )
-    (property "LCSC Part #" "C72041" (at 81.28 120.65 90)
+    (property "Vendor PN" "C72043" (at 83.82 118.11 0)
+      (effects (font (size 1.27 1.27)) hide)
+    )
+    (property "LCSC Part #" "C72043" (at 81.28 120.65 90)
       (effects (font (size 1.27 1.27)) (justify left))
     )
@@
       (effects (font (size 1.27 1.27)) (justify left))
     )
-    (property "Value" "BLUE/0603" (at 81.28 80.01 90)
+    (property "Value" "GREEN/0603" (at 81.28 80.01 90)
       (effects (font (size 1.27 1.27)) (justify left))
     )
@@
       (effects (font (size 1.27 1.27)) hide)
     )
-    (property "Mfr PN" "19-217/BHC-ZL1M2RY/3T" (at 83.82 80.01 0)
+    (property "Mfr PN" "19-217/GHC-YR1S2/3T" (at 83.82 80.01 0)
       (effects (font (size 1.27 1.27)) hide)
     )
@@
       (effects (font (size 1.27 1.27)) hide)
     )
-    (property "Vendor PN" "C72041" (at 83.82 80.01 0)
-      (effects (font (size 1.27 1.27)) hide)
-    )
-    (property "LCSC Part #" "C72041" (at 81.28 82.55 90)
+    (property "Vendor PN" "C72043" (at 83.82 80.01 0)
+      (effects (font (size 1.27 1.27)) hide)
+    )
+    (property "LCSC Part #" "C72043" (at 81.28 82.55 90)
       (effects (font (size 1.27 1.27)) (justify left))
     )
@@
       (effects (font (size 1.27 1.27)) (justify left))
     )
-    (property "Value" "BLUE/0603" (at 184.15 80.01 90)
+    (property "Value" "GREEN/0603" (at 184.15 80.01 90)
       (effects (font (size 1.27 1.27)) (justify left))
     )
@@
       (effects (font (size 1.27 1.27)) hide)
     )
-    (property "Mfr PN" "19-217/BHC-ZL1M2RY/3T" (at 186.69 80.01 0)
+    (property "Mfr PN" "19-217/GHC-YR1S2/3T" (at 186.69 80.01 0)
       (effects (font (size 1.27 1.27)) hide)
     )
@@
       (effects (font (size 1.27 1.27)) hide)
     )
-    (property "Vendor PN" "C72041" (at 186.69 80.01 0)
-      (effects (font (size 1.27 1.27)) hide)
-    )
-    (property "LCSC Part #" "C72041" (at 184.15 82.55 90)
-      (effects (font (size 1.27 1.27)) (justify left))
-    )
+    (property "Vendor PN" "C72043" (at 186.69 80.01 0)
+      (effects (font (size 1.27 1.27)) hide)
+    )
+    (property "LCSC Part #" "C72043" (at 184.15 82.55 90)
+      (effects (font (size 1.27 1.27)) (justify left))
+    )

Commit message: Redone everything
Parts:
- removed J3: OUT4, Tales:TerminalBlock_Phoenix_MKDS-3-2-5.08_1x02_P5.08mm_Horizontal, symbol Connector_Generic:Conn_01x02
- removed J3: OUT2, Tales:TerminalBlock_Phoenix_MKDS-3-2-5.08_1x02_P5.08mm_Horizontal, symbol Connector_Generic:Conn_01x02
- removed J3: OUT3, Tales:TerminalBlock_Phoenix_MKDS-3-2-5.08_1x02_P5.08mm_Horizontal, symbol Connector_Generic:Conn_01x02
- D? (x4): renamed from D14; value GREEN/0603 -> GREEN; Case 0603 -> (none); Package (none) -> 0603/1608
- D? (x4): renamed from D15; value 1N4148/SOD-123 -> 1N4148; Case SOD-123 -> (none); Package (none) -> SOD-123
- J1: value Conn_01x05 -> DG141V-2.54-6P; footprint Tales:TerminalBlock_DG141V-2.54-5P_1x05_P2.54mm_Vertical -> Tales:TerminalBlock_Dibo_DB141V-2.54-6P_1x06_P2.54mm_Vertical; symbol Connector_Generic:Conn_01x05 -> Connector_Generic:Conn_01x06; Mfr Dibo -> DIBO
- J?: renamed from J3; value OUT1 -> DB142V-5.08-8P; footprint Tales:TerminalBlock_Phoenix_MKDS-3-2-5.08_1x02_P5.08mm_Horizontal -> Tales:TerminalBlock_Dibo_DB142V-5.08-8P_1x08_P5.08mm_Vertical; symbol Connector_Generic:Conn_01x02 -> Connector_Generic:Conn_01x08; JLCPCB BOM 0 -> 1; LCSC Part # (none) -> C2898705; Mfr Metaltex -> DIBO; Mfr PN BR902V -> DB142V-5.08-8P; Vendor Eletropeças -> JLCPCB; Vendor PN 29273 -> C2898705
- K? (x4): renamed from K1; footprint Tales:Relay_SPST_Omron-G5PZ-1A -> Tales:Relay_SPST_Omron_G5PZ-1A; Technology (none) -> SPST
- R? (x4): renamed from R27; value 4k7/0,125W/0805 -> 5k6/100mW; footprint Tales:R_0805_2012Metric -> Tales:R_0603_1608Metric; Case 0805/2012 -> (none); LCSC Part # C17673 -> C23189; Package (none) -> 0603/1608; Vendor PN C17673 -> C23189
- RV? (x4): renamed from RV1; value 250VAC -> 275VAC; footprint Tales:RV_Disc_D12mm_W3.9mm_P7.5mm -> Tales:RV_Disc_D9.50mm_W3.6mm_P5.08mm; JLCPCB BOM 0 -> 1; LCSC Part # (none) -> C2761646; Mfr Yageo -> Dersonic; Mfr PN 391KD10 -> RM07D431KC1IE100; Package (none) -> 9.5X5.08mm; Vendor Mouser -> JLCPCB; Vendor PN 603-391KD10 -> C2761646
Connections:
- net +24V: now also J1.6 (Pin_6)
- net at K?.2, RV?.1: now also J?.5 (Pin_5)
- net at K?.3, RV?.2: now also J?.6 (Pin_6)
- net at K?.2, RV?.1: now also J?.7 (Pin_7)
- net at K?.3, RV?.2: now also J?.8 (Pin_8)
- net at K?.2, RV?.1: now also J?.3 (Pin_3)
- net at K?.3, RV?.2: now also J?.4 (Pin_4)
Other:
- moved on the sheet: D?, K?, R?, RV?

Commit message: Standarization
Other:
- title: 4x 24V Relay Module -> 4x 24V 12A Relay Module
Changed lines of the file:
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@@
   (paper "A4")
   (title_block
-    (title "4x 24V Relay Module")
+    (title "4x 24V 12A Relay Module")
     (date "2023-05-21")
     (rev "V1")
