File: V2/Relay-24v-4ch-V2.kicad_sch (KiCad schematic)
At the start: 25 parts, among them J1 Conn_01x05, J3 OUT1, J3 OUT2, J3 OUT3, J3 OUT4, K1 SRD-DC24V-SL-C, K2 SRD-DC24V-SL-C, K3 SRD-DC24V-SL-C, K4 SRD-DC24V-SL-C

Commit message: Input connector rotated 180deg
Parts:
- removed K1, K2, K3, K4: SRD-DC24V-SL-C, Relay_THT:Relay_SPDT_Finder_36.11, symbol Relay:FINDER-36.11
- added K1, K2, K3, K4: SRD-24VDC-SL-A, Tales:Relay_SPST_Songle_SRD_FormA, symbol Tales:Songle_SRD
- J1: value Conn_01x05 -> IN; footprint Tales:TerminalBlock_DG141V-2.54-5P_1x05_P2.54mm_Vertical -> Tales:TerminalBlock_Phoenix_FFKDSA1-V-2.54-5_1x05_P2.54mm_Vertical
- J3: footprint Tales:TerminalBlock_Phoenix_MKDS-3-2-5.08_1x02_P5.08mm_Horizontal -> Tales:TerminalBlock_Phoenix_FFKDSA-V1-5.08-2_1x02_P5.08mm_Vertical; JLCPCB BOM 0 -> 1; Vendor Eletropeças -> JLCPCB; Vendor PN 29273 -> (none)
Connections:
- net +24V: now also K1.A1, K2.A1, K3.A1, K4.A1
- net at D14.1 (K), D15.2 (A), J1.1 (Pin_1): now also K4.A2
- net at J3.2 (Pin_2), RV1.2: now also K3.11
- net at J3.1 (Pin_1), RV1.1: now also K3.14
- net at D14.1 (K), D15.2 (A), J1.2 (Pin_2): now also K3.A2
- net at D14.1 (K), D15.2 (A), J1.4 (Pin_4): now also K1.A2
- net at J3.2 (Pin_2), RV1.2: now also K2.11
- net at J3.1 (Pin_1), RV1.1: now also K2.14
- net at D14.1 (K), D15.2 (A), J1.3 (Pin_3): now also K2.A2
- net at J3.1 (Pin_1), RV1.1: now also K4.14
- net at J3.2 (Pin_2), RV1.2: now also K4.11
- net at J3.1 (Pin_1), RV1.1: now also K1.14
- net at J3.2 (Pin_2), RV1.2: now also K1.11
Other:
- moved on the sheet: J3, RV1

Commit message: Varistor updated
Parts:
- RV1: value 250VAC -> 275VAC; Mfr PN 391KD10 -> 431KD10; Vendor PN 603-391KD10 -> 603-431KD10
Changed lines of the file:
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@@
       (effects (font (size 1.27 1.27)))
     )
-    (property "Value" "250VAC" (at 245.11 100.33 0)
+    (property "Value" "275VAC" (at 245.11 100.33 0)
       (effects (font (size 1.27 1.27)))
     )
@@
       (effects (font (size 1.27 1.27)) hide)
     )
-    (property "Mfr PN" "391KD10" (at 245.11 114.3 0)
+    (property "Mfr PN" "431KD10" (at 245.11 114.3 0)
       (effects (font (size 1.27 1.27)) hide)
     )
@@
       (effects (font (size 1.27 1.27)) hide)
     )
-    (property "Vendor PN" "603-391KD10" (at 245.11 114.3 0)
+    (property "Vendor PN" "603-431KD10" (at 245.11 114.3 0)
       (effects (font (size 1.27 1.27)) hide)
     )
@@
       (effects (font (size 1.27 1.27)))
     )
-    (property "Value" "250VAC" (at 245.11 62.23 0)
+    (property "Value" "275VAC" (at 245.11 62.23 0)
       (effects (font (size 1.27 1.27)))
     )
@@
       (effects (font (size 1.27 1.27)) hide)
     )
-    (property "Mfr PN" "391KD10" (at 245.11 76.2 0)
+    (property "Mfr PN" "431KD10" (at 245.11 76.2 0)
       (effects (font (size 1.27 1.27)) hide)
     )
@@
       (effects (font (size 1.27 1.27)) hide)
     )
-    (property "Vendor PN" "603-391KD10" (at 245.11 76.2 0)
+    (property "Vendor PN" "603-431KD10" (at 245.11 76.2 0)
       (effects (font (size 1.27 1.27)) hide)
     )
@@
       (effects (font (size 1.27 1.27)))
     )
-    (property "Value" "250VAC" (at 142.24 62.23 0)
+    (property "Value" "275VAC" (at 142.24 62.23 0)
       (effects (font (size 1.27 1.27)))
     )
@@
       (effects (font (size 1.27 1.27)) hide)
     )
-    (property "Mfr PN" "391KD10" (at 142.24 76.2 0)
+    (property "Mfr PN" "431KD10" (at 142.24 76.2 0)
       (effects (font (size 1.27 1.27)) hide)
     )
@@
       (effects (font (size 1.27 1.27)) hide)
     )
-    (property "Vendor PN" "603-391KD10" (at 142.24 76.2 0)
+    (property "Vendor PN" "603-431KD10" (at 142.24 76.2 0)
       (effects (font (size 1.27 1.27)) hide)
     )
@@
       (effects (font (size 1.27 1.27)))
     )
-    (property "Value" "250VAC" (at 142.24 100.33 0)
+    (property "Value" "275VAC" (at 142.24 100.33 0)
       (effects (font (size 1.27 1.27)))
     )
@@
       (effects (font (size 1.27 1.27)) hide)
     )
-    (property "Mfr PN" "391KD10" (at 142.24 114.3 0)
+    (property "Mfr PN" "431KD10" (at 142.24 114.3 0)
       (effects (font (size 1.27 1.27)) hide)
     )
@@
       (effects (font (size 1.27 1.27)) hide)
     )
-    (property "Vendor PN" "603-391KD10" (at 142.24 114.3 0)
-      (effects (font (size 1.27 1.27)) hide)
-    )
+    (property "Vendor PN" "603-431KD10" (at 142.24 114.3 0)
+      (effects (font (size 1.27 1.27)) hide)
+    )

Commit message: Design optimization
Parts:
- J1: value IN -> DB141V-2.54-5P; footprint Tales:TerminalBlock_Phoenix_FFKDSA1-V-2.54-5_1x05_P2.54mm_Vertical -> Tales:TerminalBlock_Dibo_DB141V-2.54-5P_1x05_P2.54mm_Vertical
- J3: value OUT4 -> DB142V-5.08-2P; footprint Tales:TerminalBlock_Phoenix_FFKDSA-V1-5.08-2_1x02_P5.08mm_Vertical -> Tales:TerminalBlock_Dibo_DB142V-5.08-2P_1x02_P5.08mm_Vertical; Mfr Metaltex -> (none); Mfr PN BR902V -> (none)
- J3: value OUT2 -> DB142V-5.08-2P; footprint Tales:TerminalBlock_Phoenix_FFKDSA-V1-5.08-2_1x02_P5.08mm_Vertical -> Tales:TerminalBlock_Dibo_DB142V-5.08-2P_1x02_P5.08mm_Vertical; Mfr Metaltex -> (none); Mfr PN BR902V -> (none)
- J3: value OUT1 -> DB142V-5.08-2P; footprint Tales:TerminalBlock_Phoenix_FFKDSA-V1-5.08-2_1x02_P5.08mm_Vertical -> Tales:TerminalBlock_Dibo_DB142V-5.08-2P_1x02_P5.08mm_Vertical; Mfr Metaltex -> (none); Mfr PN BR902V -> (none)
- J3: value OUT3 -> DB142V-5.08-2P; footprint Tales:TerminalBlock_Phoenix_FFKDSA-V1-5.08-2_1x02_P5.08mm_Vertical -> Tales:TerminalBlock_Dibo_DB142V-5.08-2P_1x02_P5.08mm_Vertical; Mfr Metaltex -> (none); Mfr PN BR902V -> (none)
- RV1: footprint Tales:RV_Disc_D12mm_W3.9mm_P7.5mm -> Tales:RV_Disc_D9.50mm_W3.6mm_P5.08mm
Changed lines of the file:
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@@
-      (effects (font (size 1.27 1.27)) hide)
-    )
-    (property "Sim.Device" "D" (at 92.71 74.93 0)
-      (effects (font (size 1.27 1.27)) hide)
-    )
-    (property "Sim.Pins" "1=K 2=A" (at 92.71 74.93 0)
       (effects (font (size 1.27 1.27)) hide)
     )
@@
       (effects (font (size 1.27 1.27)))
     )
-    (property "Value" "IN" (at 38.1 80.01 0)
-      (effects (font (size 1.27 1.27)))
-    )
-    (property "Footprint" "Tales:TerminalBlock_Phoenix_FFKDSA1-V-2.54-5_1x05_P2.54mm_Vertical" (at 38.1 88.9 0)
+    (property "Value" "DB141V-2.54-5P" (at 38.1 80.01 0)
+      (effects (font (size 1.27 1.27)))
+    )
+    (property "Footprint" "Tales:TerminalBlock_Dibo_DB141V-2.54-5P_1x05_P2.54mm_Vertical" (at 38.1 88.9 0)
       (effects (font (size 1.27 1.27)) hide)
     )
@@
       (effects (font (size 1.27 1.27)))
     )
-    (property "Value" "OUT4" (at 262.89 109.22 0)
-      (effects (font (size 1.27 1.27)))
-    )
-    (property "Footprint" "Tales:TerminalBlock_Phoenix_FFKDSA-V1-5.08-2_1x02_P5.08mm_Vertical" (at 259.08 104.14 0)
+    (property "Value" "DB142V-5.08-2P" (at 262.89 109.22 0)
+      (effects (font (size 1.27 1.27)))
+    )
+    (property "Footprint" "Tales:TerminalBlock_Dibo_DB142V-5.08-2P_1x02_P5.08mm_Vertical" (at 259.08 104.14 0)
       (effects (font (size 1.27 1.27)) hide)
     )
@@
       (effects (font (size 1.27 1.27)) hide)
     )
-    (property "Mfr" "Metaltex" (at 259.08 104.14 0)
-      (effects (font (size 1.27 1.27)) hide)
-    )
-    (property "Mfr PN" "BR902V" (at 259.08 104.14 0)
+    (property "Mfr" "" (at 259.08 104.14 0)
+      (effects (font (size 1.27 1.27)) hide)
+    )
+    (property "Mfr PN" "" (at 259.08 104.14 0)
       (effects (font (size 1.27 1.27)) hide)
     )
@@
       (effects (font (size 1.27 1.27)))
     )
-    (property "Value" "OUT2" (at 262.89 71.12 0)
-      (effects (font (size 1.27 1.27)))
-    )
-    (property "Footprint" "Tales:TerminalBlock_Phoenix_FFKDSA-V1-5.08-2_1x02_P5.08mm_Vertical" (at 259.08 66.04 0)
+    (property "Value" "DB142V-5.08-2P" (at 262.89 71.12 0)
+      (effects (font (size 1.27 1.27)))
+    )
+    (property "Footprint" "Tales:TerminalBlock_Dibo_DB142V-5.08-2P_1x02_P5.08mm_Vertical" (at 259.08 66.04 0)
       (effects (font (size 1.27 1.27)) hide)
     )
@@
       (effects (font (size 1.27 1.27)) hide)
     )
-    (property "Mfr" "Metaltex" (at 259.08 66.04 0)
-      (effects (font (size 1.27 1.27)) hide)
-    )
-    (property "Mfr PN" "BR902V" (at 259.08 66.04 0)
+    (property "Mfr" "" (at 259.08 66.04 0)
+      (effects (font (size 1.27 1.27)) hide)
+    )
+    (property "Mfr PN" "" (at 259.08 66.04 0)
       (effects (font (size 1.27 1.27)) hide)
     )
@@
       (effects (font (size 1.27 1.27)))
     )
-    (property "Footprint" "Tales:RV_Disc_D12mm_W3.9mm_P7.5mm" (at 243.332 114.3 90)
+    (property "Footprint" "Tales:RV_Disc_D9.50mm_W3.6mm_P5.08mm" (at 243.332 114.3 90)
       (effects (font (size 1.27 1.27)) hide)
     )
@@
       (effects (font (size 1.27 1.27)))
     )
-    (property "Footprint" "Tales:RV_Disc_D12mm_W3.9mm_P7.5mm" (at 243.332 76.2 90)
+    (property "Footprint" "Tales:RV_Disc_D9.50mm_W3.6mm_P5.08mm" (at 243.332 76.2 90)
       (effects (font (size 1.27 1.27)) hide)
     )
@@
       (effects (font (size 1.27 1.27)))
     )
-    (property "Value" "OUT1" (at 160.02 71.12 0)
-      (effects (font (size 1.27 1.27)))
-    )
-    (property "Footprint" "Tales:TerminalBlock_Phoenix_FFKDSA-V1-5.08-2_1x02_P5.08mm_Vertical" (at 156.21 66.04 0)
+    (property "Value" "DB142V-5.08-2P" (at 160.02 71.12 0)
+      (effects (font (size 1.27 1.27)))
+    )
+    (property "Footprint" "Tales:TerminalBlock_Dibo_DB142V-5.08-2P_1x02_P5.08mm_Vertical" (at 156.21 66.04 0)
       (effects (font (size 1.27 1.27)) hide)
     )
@@
       (effects (font (size 1.27 1.27)) hide)
     )
-    (property "Mfr" "Metaltex" (at 156.21 66.04 0)
-      (effects (font (size 1.27 1.27)) hide)
-    )
-    (property "Mfr PN" "BR902V" (at 156.21 66.04 0)
+    (property "Mfr" "" (at 156.21 66.04 0)
+      (effects (font (size 1.27 1.27)) hide)
+    )
+    (property "Mfr PN" "" (at 156.21 66.04 0)
       (effects (font (size 1.27 1.27)) hide)
     )
@@
       (effects (font (size 1.27 1.27)))
     )
-    (property "Value" "OUT3" (at 160.02 109.22 0)
-      (effects (font (size 1.27 1.27)))
-    )
-    (property "Footprint" "Tales:TerminalBlock_Phoenix_FFKDSA-V1-5.08-2_1x02_P5.08mm_Vertical" (at 156.21 104.14 0)
+    (property "Value" "DB142V-5.08-2P" (at 160.02 109.22 0)
+      (effects (font (size 1.27 1.27)))
+    )
+    (property "Footprint" "Tales:TerminalBlock_Dibo_DB142V-5.08-2P_1x02_P5.08mm_Vertical" (at 156.21 104.14 0)
       (effects (font (size 1.27 1.27)) hide)
     )
@@
       (effects (font (size 1.27 1.27)) hide)
     )
-    (property "Mfr" "Metaltex" (at 156.21 104.14 0)
-      (effects (font (size 1.27 1.27)) hide)
-    )
-    (property "Mfr PN" "BR902V" (at 156.21 104.14 0)
+    (property "Mfr" "" (at 156.21 104.14 0)
+      (effects (font (size 1.27 1.27)) hide)
+    )
+    (property "Mfr PN" "" (at 156.21 104.14 0)
       (effects (font (size 1.27 1.27)) hide)
     )
@@
       (effects (font (size 1.27 1.27)) hide)
     )
-    (property "Sim.Device" "D" (at 195.58 113.03 0)
-      (effects (font (size 1.27 1.27)) hide)
-    )
-    (property "Sim.Pins" "1=K 2=A" (at 195.58 113.03 0)
-      (effects (font (size 1.27 1.27)) hide)
-    )
     (pin "1")
     (pin "2")
@@
       (effects (font (size 1.27 1.27)) hide)
     )
-    (property "Sim.Device" "D" (at 92.71 113.03 0)
-      (effects (font (size 1.27 1.27)) hide)
-    )
-    (property "Sim.Pins" "1=K 2=A" (at 92.71 113.03 0)
-      (effects (font (size 1.27 1.27)) hide)
-    )
     (pin "1")
     (pin "2")
@@
       (effects (font (size 1.27 1.27)) hide)
     )
-    (property "Sim.Device" "D" (at 195.58 74.93 0)
-      (effects (font (size 1.27 1.27)) hide)
-    )
-    (property "Sim.Pins" "1=K 2=A" (at 195.58 74.93 0)
-      (effects (font (size 1.27 1.27)) hide)
-    )
     (pin "1")
     (pin "2")
@@
       (effects (font (size 1.27 1.27)))
     )
-    (property "Footprint" "Tales:RV_Disc_D12mm_W3.9mm_P7.5mm" (at 140.462 76.2 90)
+    (property "Footprint" "Tales:RV_Disc_D9.50mm_W3.6mm_P5.08mm" (at 140.462 76.2 90)
       (effects (font (size 1.27 1.27)) hide)
     )
@@
       (effects (font (size 1.27 1.27)))
     )
-    (property "Footprint" "Tales:RV_Disc_D12mm_W3.9mm_P7.5mm" (at 140.462 114.3 90)
-      (effects (font (size 1.27 1.27)) hide)
-    )
+    (property "Footprint" "Tales:RV_Disc_D9.50mm_W3.6mm_P5.08mm" (at 140.462 114.3 90)
+      (effects (font (size 1.27 1.27)) hide)
+    )

Commit message: Redone everything
Parts:
- removed J3 (x3): DB142V-5.08-2P, Tales:TerminalBlock_Dibo_DB142V-5.08-2P_1x02_P5.08mm_Vertical, symbol Connector_Generic:Conn_01x02
- removed K1, K2, K3, K4: SRD-24VDC-SL-A, Tales:Relay_SPST_Songle_SRD_FormA, symbol Tales:Songle_SRD
- added K? (x4): G5Q-1A4-DC24V, Tales:Relay_SPST_Omron-G5Q-1A, symbol Tales:G5Q-1A
- D? (x4): renamed from D14; value GREEN/0603 -> GREEN; Case 0603 -> (none); Package (none) -> 0603/1608
- D? (x4): renamed from D15; value 1N4148/SOD-123 -> 1N4148; Case SOD-123 -> (none); Package (none) -> SOD-123
- J1: value DB141V-2.54-5P -> DG141V-2.54-6P; footprint Tales:TerminalBlock_Dibo_DB141V-2.54-5P_1x05_P2.54mm_Vertical -> Tales:TerminalBlock_Dibo_DB141V-2.54-6P_1x06_P2.54mm_Vertical; symbol Connector_Generic:Conn_01x05 -> Connector_Generic:Conn_01x06; Mfr Dibo -> DIBO
- J?: renamed from J3; value DB142V-5.08-2P -> DB142V-5.08-8P; footprint Tales:TerminalBlock_Dibo_DB142V-5.08-2P_1x02_P5.08mm_Vertical -> Tales:TerminalBlock_Dibo_DB142V-5.08-8P_1x08_P5.08mm_Vertical; symbol Connector_Generic:Conn_01x02 -> Connector_Generic:Conn_01x08; LCSC Part # (none) -> C2898705; Mfr (none) -> DIBO; Mfr PN (none) -> DB142V-5.08-8P; Vendor PN (none) -> C2898705
- R? (x4): renamed from R27; value 4k7/0,125W/0805 -> 5k6/100mW; footprint Tales:R_0805_2012Metric -> Tales:R_0603_1608Metric; Case 0805/2012 -> (none); LCSC Part # C17673 -> C23189; Package (none) -> 0603/1608; Vendor PN C17673 -> C23189
- RV? (x4): renamed from RV1; JLCPCB BOM 0 -> 1; LCSC Part # (none) -> C2761646; Mfr Yageo -> Dersonic; Mfr PN 431KD10 -> RM07D431KC1IE100; Package (none) -> 9.5X5.08mm; Vendor Mouser -> JLCPCB; Vendor PN 603-431KD10 -> C2761646
Connections:
- net +24V: now also J1.6 (Pin_6), K?.1, K?.1, K?.1, K?.1
- net at D?.1 (K), D?.2 (A), J1.1 (Pin_1): now also K?.5
- net at D?.1 (K), D?.2 (A), J1.4 (Pin_4): now also K?.5
- net at D?.1 (K), D?.2 (A), J1.2 (Pin_2): now also K?.5
- net at D?.1 (K), D?.2 (A), J1.3 (Pin_3): now also K?.5
- net at RV?.1: now also J?.7 (Pin_7), K?.3
- net at RV?.2: now also J?.8 (Pin_8), K?.2
- net at RV?.1: now also J?.3 (Pin_3), K?.3
- net at RV?.2: now also J?.4 (Pin_4), K?.2
- net at J?.1 (Pin_1), RV?.1: now also K?.3
- net at J?.2 (Pin_2), RV?.2: now also K?.2
- net at RV?.1: now also J?.5 (Pin_5), K?.3
- net at RV?.2: now also J?.6 (Pin_6), K?.2
Other:
- moved on the sheet: D?, R?, RV?

Commit message: Standarization
Other:
- title: 4x 24V Relay Module -> 4x 24V 8A Relay Module
Changed lines of the file:
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@@
   (paper "A4")
   (title_block
-    (title "4x 24V Relay Module")
+    (title "4x 24V 8A Relay Module")
     (date "2023-05-21")
     (rev "V1")
